File: kicad-power-src-scheme/germanium-power-src.kicad_pcb (KiCad board)
At the start: 2 copper layers, 60 x 51 mm, 17 parts, among them J1 Вход, J2 П213, J3 Вых, Q1 MP42

Commit message: Add files via upload
Parts:
- D1, D2, D7: value Д223 -> Д9
- D3, D4, D5, D6: value Д2 -> Д7
Changed lines of the file:
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@@
         (effects (font (size 1 1) (thickness 0.15)))
     )
-    (fp_text value "Д2" (at 6.35 0.2) (layer "F.SilkS")
+    (fp_text value "Д7" (at 6.35 0.2) (layer "F.SilkS")
         (effects (font (size 1 1) (thickness 0.15)))
     )
@@
         (effects (font (size 1 1) (thickness 0.15)))
     )
-    (fp_text value "Д2" (at 6.7 0.1) (layer "F.SilkS")
+    (fp_text value "Д7" (at 6.7 0.1) (layer "F.SilkS")
         (effects (font (size 1 1) (thickness 0.15)))
     )
@@
         (effects (font (size 1 1) (thickness 0.15)))
     )
-    (fp_text value "Д223" (at 5.1 2.8 90) (layer "F.SilkS")
+    (fp_text value "Д9" (at 5.1 2.8 90) (layer "F.SilkS")
         (effects (font (size 1 1) (thickness 0.15)))
     )
@@
         (effects (font (size 1 1) (thickness 0.15)))
     )
-    (fp_text value "Д2" (at 6.5 0.2) (layer "F.SilkS")
+    (fp_text value "Д7" (at 6.5 0.2) (layer "F.SilkS")
         (effects (font (size 1 1) (thickness 0.15)))
     )
@@
         (effects (font (size 1 1) (thickness 0.15)))
     )
-    (fp_text value "Д223" (at 14.3 0 90) (layer "F.SilkS")
+    (fp_text value "Д9" (at 14.3 0 90) (layer "F.SilkS")
         (effects (font (size 1 1) (thickness 0.15)))
     )
@@
         (effects (font (size 1 1) (thickness 0.15)))
     )
-    (fp_text value "Д223" (at 5.3 2.9 90) (layer "F.SilkS")
+    (fp_text value "Д9" (at 5.3 2.9 90) (layer "F.SilkS")
         (effects (font (size 1 1) (thickness 0.15)))
     )
@@
         (effects (font (size 1 1) (thickness 0.15)))
     )
-    (fp_text value "Д2" (at 6.6 0) (layer "F.SilkS")
-        (effects (font (size 1 1) (thickness 0.15)))
-    )
+    (fp_text value "Д7" (at 6.6 0) (layer "F.SilkS")
+        (effects (font (size 1 1) (thickness 0.15)))
+    )

Commit message: Migrate to KiCad 8.0
Parts:
- C1: value 470Mф 15В -> 470MФ 15B
- J1: value Вход -> Bxoд
- Q1: value MP42 -> MП42
- RV1: value 10K Рег -> 10K
- Д7: renamed from D3; value Д7 -> D224
- Д7: renamed from D4; value Д7 -> D224
- Д9: renamed from D1; value Д9 -> D224; footprint Soviet:D223 -> Soviet:D9
- Д9: renamed from D2; value Д9 -> D224; footprint Soviet:D223 -> Soviet:D9
- Д9: renamed from D7; value Д9 -> D224; footprint Soviet:D223 -> Soviet:D9
- moved D5 20.0 mm to (129.5, 95.5), turned to 180 degrees
- moved Д7 20.0 mm to (129.5, 83.5), turned to 180 degrees
Routing:
- net Net-(D3-K): track 53.1 -> 26.9 mm
- net Net-(D4-K): track 50.2 -> 33.6 mm
- net +12V: track 64.9 -> 80.3 mm
- net Net-(J2-Pin_2): track 38.0 -> 34.3 mm
- net Net-(J2-Pin_1): track 33.2 -> 35.8 mm
- net -12V: track 70.2 -> 69.6 mm

Commit message: Minor fixes
Parts:
- renumbered Д9 to Д814

Commit message: Minor fixes
Parts:
- removed Д7 (x2): D224, Soviet:D2
- removed Д814 (x3): D224, Soviet:D9
- added C2: 470Mф 15В, Capacitor_THT:CP_Radial_D10.0mm_P3.50mm, F.Cu at (140.0, 88.0)
- added C3: 100n, Capacitor_THT:C_Axial_L3.8mm_D2.6mm_P7.50mm_Horizontal, F.Cu at (146.5, 95.5)
- added C4: 100n, Capacitor_THT:C_Axial_L3.8mm_D2.6mm_P7.50mm_Horizontal, F.Cu at (115.0, 84.0)
- added C5: 100n, Capacitor_THT:C_Axial_L3.8mm_D2.6mm_P7.50mm_Horizontal, F.Cu at (115.0, 95.0)
- added C6: 100n, Capacitor_THT:C_Axial_L3.8mm_D2.6mm_P7.50mm_Horizontal, F.Cu at (115.0, 117.0)
- added C7: 100n, Capacitor_THT:C_Axial_L3.8mm_D2.6mm_P7.50mm_Horizontal, F.Cu at (122.5, 106.0)
- added D3: Д7, Soviet:D7, F.Cu at (108.1, 100.5)
- added D4: Д7, Soviet:D7, F.Cu at (129.9, 111.5)
- added DZ1: Стаб 10В, Diode_THT:D_DO-15_P12.70mm_Horizontal, F.Cu at (148.5, 120.5)
- added J4: Конд Вых, Connector_PinSocket_2.54mm:PinSocket_1x02_P2.54mm_Vertical, F.Cu at (156.0, 105.5)
- added Strogg logo: Strogg_logo, Symbol:Strogg_logo, F.Cu at (148.5, 101.5)
- C1: value 470MФ 15B -> 470Mф 15В
- D5, D6: footprint Soviet:D2 -> Soviet:D7
- G***: value LOGO -> LOGO CCCP; footprint LOGO -> Soviet:LOGO CCCP
- J1: value Bxoд -> Вход
- J2: value П213 -> П214
- J3: value Вых -> Выход
- moved RV1 27.8 mm to (141.0, 96.5), turned to 0 degrees
- moved D5 27.0 mm to (108.5, 78.5), turned to 0 degrees
- moved R2 25.7 mm to (102.0, 92.1), turned to 90 degrees
- moved R1 25.1 mm to (144.1, 105.0), turned to 180 degrees
- moved D6 23.7 mm to (129.9, 89.5), turned to 180 degrees
- moved R3 21.8 mm to (102.0, 94.8), turned to -90 degrees
- moved C1 14.6 mm to (148.2, 88.0)
- moved J3 14.1 mm to (146.0, 76.0), turned to 90 degrees
- moved J2 12.8 mm to (140.5, 76.0), turned to -90 degrees
- moved J1 7.92 mm to (102.0, 111.5), turned to 180 degrees
- moved Q1 7.52 mm to (135.9, 116.5)
- moved G*** 0.51 mm to (109.5, 119.5)
Connections:
- D5 pad 1: -12V -> Net-(D4-A)
- D5 pad 2: Net-(D4-K) -> -12V
- D6 pad 1: -12V -> Net-(D3-A)
- D6 pad 2: Net-(D3-K) -> -12V
- J1 pad 1: Net-(D3-K) -> Net-(D3-A)
- J1 pad 2: Net-(D4-K) -> Net-(D4-A)
Routing:
- net -12V: track 69.6 -> 0.00 mm
- net Net-(D4-A): track 0.00 -> 68.2 mm
- net +12V: track 80.3 -> 142.5 mm
- net Net-(D3-A): track 0.00 -> 56.3 mm
- net Net-(J2-Pin_1): track 35.8 -> 91.8 mm
- net Net-(J2-Pin_2): track 34.3 -> 80.4 mm
- net Net-(D4-K): track 33.6 -> 0.00 mm
- net Net-(D3-K): track 26.9 -> 0.00 mm
- net Net-(DZ1-A): track 37.2 -> 26.4 mm
- net Net-(Q1-B): track 24.4 -> 18.1 mm
- net Net-(D2-A): track 4.00 -> 0.00 mm
- net Net-(D1-K): track 3.50 -> 0.00 mm
