File: kicad-power-src-scheme/germanium-power-src.kicad_sch (KiCad schematic)
At the start: 16 parts, among them J2 P213, J4 In, J4 Out, Q1 MP42

Commit message: Migrate to KiCad 8.0
Parts:
- D1: footprint Soviet:D223 -> Soviet:D9; symbol Soviet:D223 -> Soviet:D9

Commit message: Minor fixes
Parts:
- D1: symbol Soviet:D9 -> PCM_Diode_Zener_AKL:D_Zener_Generic
Connections:
- net +12V: now also D1.1 (K); no longer D1.2 (K)
- net at D1.2 (A): now also D1.1 (K); no longer D1.1 (A)
- net at D1.1 (K): now also D1.2 (A); no longer D1.2 (K)
- net at R4.1, RV1.1: now also D1.2 (A); no longer D1.1 (A)
Changed lines of the file:
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@@
 	)
 	(symbol
-		(lib_id "Soviet:D9")
+		(lib_id "PCM_Diode_Zener_AKL:D_Zener_Generic")
 		(at 58.42 162.56 270)
 		(unit 1)
@@
 		(fields_autoplaced yes)
 		(property "Reference" "D1"
-			(at 60.96 161.925 90)
+			(at 60.96 161.2899 90)
 			(effects
 				(font
@@
 		)
 		(property "Value" "D224"
-			(at 60.96 164.465 90)
+			(at 60.96 163.8299 90)
 			(effects
 				(font
@@
 		)
 		(property "Footprint" "Soviet:D9"
-			(at 49.53 162.56 0)
-			(effects
-				(font
-					(size 1.27 1.27)
-				)
-				(hide yes)
-			)
-		)
-		(property "Datasheet" "https://static.chipdip.ru/lib/270/DOC000270836.pdf"
-			(at 52.07 161.29 0)
-			(effects
-				(font
-					(size 1.27 1.27)
-				)
-				(hide yes)
-			)
-		)
-		(property "Description" ""
+			(at 58.42 162.56 0)
+			(effects
+				(font
+					(size 1.27 1.27)
+				)
+				(hide yes)
+			)
+		)
+		(property "Datasheet" "~"
+			(at 58.42 162.56 0)
+			(effects
+				(font
+					(size 1.27 1.27)
+				)
+				(hide yes)
+			)
+		)
+		(property "Description" "Zener diode, generic symbol, Alternate KiCAD Library"
 			(at 58.42 162.56 0)
 			(effects
@@
 	)
 	(symbol
-		(lib_id "Soviet:D9")
+		(lib_id "PCM_Diode_Zener_AKL:D_Zener_Generic")
 		(at 58.42 152.4 270)
 		(unit 1)
@@
 		(fields_autoplaced yes)
 		(property "Reference" "D1"
-			(at 60.96 151.765 90)
+			(at 60.96 151.1299 90)
 			(effects
 				(font
@@
 		)
 		(property "Value" "D224"
-			(at 60.96 154.305 90)
+			(at 60.96 153.6699 90)
 			(effects
 				(font
@@
 		)
 		(property "Footprint" "Soviet:D9"
-			(at 49.53 152.4 0)
-			(effects
-				(font
-					(size 1.27 1.27)
-				)
-				(hide yes)
-			)
-		)
-		(property "Datasheet" "https://static.chipdip.ru/lib/270/DOC000270836.pdf"
-			(at 52.07 151.13 0)
-			(effects
-				(font
-					(size 1.27 1.27)
-				)
-				(hide yes)
-			)
-		)
-		(property "Description" ""
+			(at 58.42 152.4 0)
+			(effects
+				(font
+					(size 1.27 1.27)
+				)
+				(hide yes)
+			)
+		)
+		(property "Datasheet" "~"
+			(at 58.42 152.4 0)
+			(effects
+				(font
+					(size 1.27 1.27)
+				)
+				(hide yes)
+			)
+		)
+		(property "Description" "Zener diode, generic symbol, Alternate KiCAD Library"
 			(at 58.42 152.4 0)
 			(effects
@@
 	)
 	(symbol
-		(lib_id "Soviet:D9")
+		(lib_id "PCM_Diode_Zener_AKL:D_Zener_Generic")
 		(at 58.42 142.24 270)
 		(unit 1)
@@
 		(fields_autoplaced yes)
 		(property "Reference" "D1"
-			(at 60.96 141.605 90)
+			(at 60.96 140.9699 90)
 			(effects
 				(font
@@
 		)
 		(property "Value" "D224"
-			(at 60.96 144.145 90)
+			(at 60.96 143.5099 90)
 			(effects
 				(font
@@
 		)
 		(property "Footprint" "Soviet:D9"
-			(at 49.53 142.24 0)
-			(effects
-				(font
-					(size 1.27 1.27)
-				)
-				(hide yes)
-			)
-		)
-		(property "Datasheet" "https://static.chipdip.ru/lib/270/DOC000270836.pdf"
-			(at 52.07 140.97 0)
-			(effects
-				(font
-					(size 1.27 1.27)
-				)
-				(hide yes)
-			)
-		)
-		(property "Description" ""
 			(at 58.42 142.24 0)
 			(effects
+				(font
+					(size 1.27 1.27)
+				)
+				(hide yes)
+			)
+		)
+		(property "Datasheet" "~"
+			(at 58.42 142.24 0)
+			(effects
+				(font
+					(size 1.27 1.27)
+				)
+				(hide yes)
+			)
+		)
+		(property "Description" "Zener diode, generic symbol, Alternate KiCAD Library"
+			(at 58.42 142.24 0)
+			(effects

Commit message: Minor fixes
Parts:
- removed D1 (x3): D224, Soviet:D9, symbol PCM_Diode_Zener_AKL:D_Zener_Generic
- added C2: 470Mf 15V, Capacitor_THT:CP_Radial_D8.0mm_P3.50mm, symbol Device:C_Polarized
- added C3, C4, C5, C6, C7: 0.1Mf, Capacitor_THT:C_Axial_L3.8mm_D2.6mm_P7.50mm_Horizontal, symbol Device:C
- added DZ1: D_Zener_Generic, Diode_THT:D_DO-27_P12.70mm_Horizontal, symbol PCM_Diode_Zener_AKL:D_Zener_Generic
- added J4: Cap, Connector_PinSocket_2.54mm:PinSocket_1x02_P2.54mm_Vertical, symbol Connector:Conn_01x02_Pin
- D1: footprint Soviet:D2 -> Soviet:D7; symbol Soviet:D2 -> Soviet:D7
Connections:
- net +12V: now also D1.1 (K), D1.1 (K), C2.1, C3.1, C4.1, C5.2, DZ1.1 (K), J4.1 (Pin_1); no longer D1.2 (A), D1.2 (A)
- net -12V: now also D1.2 (A), D1.2 (A), C6.1, C7.2; no longer D1.1 (K), D1.1 (K)
- net at J2.1 (Pin_1), J4.2 (Pin_2), R4.2: now also C3.2, J4.2 (Pin_2)
- net at R4.1, RV1.1: now also C2.2, DZ1.2 (A)
- new net: C4.2, C7.1, D1.1 (K), D1.2 (A), J4.2 (Pin_2)
- new net: C5.1, C6.2, D1.1 (K), D1.2 (A), J4.1 (Pin_1)
Other:
- moved on the sheet: D1
